File: project/LaunchController1.kicad_sch (KiCad schematic)
At the start: 26 parts, among them J1 1729128, J2 CB2B-XH-AM, J3 B2B-XH-AM, Q1 BJT_PNP, Q2 BJT_PNP, SW1 ANT11SF1CQE

Commit message: Feat: increased PTC current rating, dropped R5 to ensure saturation on Q2
Also switched all parts (except the battery case) to a KiCad library part to update. Moving the design to KiCad (r.i.p Eagle).

Increased current rating of PTC1 to 2.5A hold, 5A trip to reduce possibility of inadvertent tripping.
Dropped R5 to ensure saturation on Q2
Q2 is surprisingly able to handle the pulse current. Peak pulse is 6A, which should cover requirement. Maybe consider ZTX618 instead, which has a higher amp rating.
Q2 (ZTX718) is being retired, so if you're reading this you need to pick a different part.
Parts:
- removed J2: CB2B-XH-AM, Connector_JST:JST_XH_B2B-XH-AM_1x02_P2.50mm_Vertical, symbol Connector:Conn_01x02_Pin
- removed J3: B2B-XH-AM, Connector_JST:JST_XH_B2B-XH-AM_1x02_P2.50mm_Vertical, symbol Connector:Conn_01x02_Pin
- removed Q1, Q2: BJT_PNP, LaunchController1:TO92-, symbol LaunchController1-eagle-import:BJT_PNP
- removed SW1: ANT11SF1CQE, LaunchController1:ANT11SF1CQE, symbol LaunchController1-eagle-import:ANT11SF1CQE
- added Q1, Q2: ZTX718, Package_TO_SOT_THT:TO-92_Inline, symbol Transistor_BJT:BC636
- added SW2, SW3, SW4: B2B-XH-AM, Connector_JST:JST_XH_B2B-XH-AM_1x02_P2.50mm_Vertical, symbol Switch:SW_SPST
- D1, D2: value P6KE75CA -> P6KE7.5CA/B; footprint LaunchController1:DIOAD1300W80L670D310 -> Diode_THT:D_DO-15_P12.70mm_Horizontal
- PTC1: value 0ZRG0120FF2E -> 0ZRG0250FF1E; footprint LaunchController1:0ZRG -> Fuse:Fuse_BelFuse_0ZRE0012FF_L8.3mm_W3.8mm
- R5: value 300 -> 100
Connections:
- net GND: now also BT1.N (NEG), D1.A, D2.A, D3.1 (K), D4.1 (K), J1.2 (Pin_2), SW2.1 (A)
- net arm: now also SW2.2 (B), SW3.1 (A)
- net launch: now also SW3.2 (B)
- net at R4.1: now also Q1.2 (C)
- net battery: now reaches BT1.P (POS)
- net battery: now also SW4.1 (A)
- net safed_power: now reaches D1.C, PTC1.2, R1.2, R2.2, R6.1, R7.2, R8.1
- net safed_power: now also Q1.1 (E), Q2.1 (E)
- net igniter_hot: now reaches D2.C, J1.1 (Pin_1), R2.1, R3.1
- net igniter_hot: now also Q2.2 (C)
- net at R3.2: now also Q1.3 (B)
- net at R5.2, R6.2: now also Q2.3 (B)
- net at PTC1.1: now also SW4.2 (B)
Other:
- moved on the sheet: D1, D2, D3, PTC1, R1, R3, R6

Commit message: Feat: Swapped Q2 from PNP BJT to PMOS
Wasn't feeling great about how close the peak pulse requirement of the BJT was to the theoretical maximum current pulse. Also didn't like the current required to put BJT into saturation. Swapped for AOD413A PMOS. Also changed resistors to accommodate PMOS gate drive.

Schematic is done, need to lay out.
Parts:
- removed Q2: ZTX718, Package_TO_SOT_THT:TO-92_Inline, symbol Transistor_BJT:BC636
- removed R5: 100, Resistor_THT:R_Axial_DIN0309_L9.0mm_D3.2mm_P12.70mm_Horizontal, symbol LaunchController1-eagle-import:RES_0.5W_TH
- added Q2: AOD413A, Package_TO_SOT_SMD:TO-252-3_TabPin2, symbol Transistor_FET:Q_PMOS_GDS
- added R9: 60, Resistor_THT:R_Axial_DIN0309_L9.0mm_D3.2mm_P12.70mm_Horizontal, symbol LaunchController1-eagle-import:RES_0.5W_TH
- D1, D2: value P6KE7.5CA/B -> P6KE7.5A/B
Connections:
- net igniter_hot: now also Q2.2 (D)
- net launch: now also R6.2, Q2.1 (G), R9.2; no longer SW3.2 (B)
- net safed_power: now also Q2.3 (S)
- new net: R9.1, SW3.2 (B)
Other:
- moved on the sheet: C1

Commit message: layout: Updated layout for schematic
Rev -
Parts:
- removed BT1: 6V, LaunchController1:BAT_2477, symbol LaunchController1-eagle-import:2477
- added J2: XT30PW-M, Connector_AMASS:AMASS_XT30PW-M_1x02_P2.50mm_Horizontal, symbol Connector:Conn_01x02_Pin
- added J3: B2B-XH-AM, Connector_JST:JST_XH_B2B-XH-AM_1x02_P2.50mm_Vertical, symbol Connector:Conn_01x02_Pin
- added TP1: TestPoint, TestPoint:TestPoint_Pad_2.0x2.0mm, symbol Connector:TestPoint
Connections:
- net GND: now also D1.2, D2.2, J2.2 (Pin_2), J3.2 (Pin_2); no longer D1.A, D2.A
- net battery: now also J2.1 (Pin_1), J3.1 (Pin_1)
- net igniter_hot: now also D2.1; no longer D2.C
- net safed_power: now also D1.1, TP1.1; no longer D1.C
Other:
- note added: "-"
- note added: "2026-08-06"
- note added: "Battery Connection"
- note added: "JGM"
- note added: "Model Rocket Launch Controller"
- note removed: "${DOCUMENT_NUMBER}"
