File: 2_Electrical/r02_launch-controller/r02_launch-controller.kicad_sch (KiCad schematic)
At the start: 32 parts, among them J1 1729128, J2 XT30PW-M, J3 B2B-XH-AM, J4 1725698, J5 1725698, Q2 BC807W, SW2 B2B-XH-AM, SW3 B2B-XH-AM, SW4 B2B-XH-AM

Commit message: layout: Laid out Rev A
Should be ready for a prototype. Same form factor as before, but all surface mount now.
Parts:
- added J6: Screw_Terminal_01x02, TerminalBlock_Phoenix:TerminalBlock_Phoenix_MPT-0,5-2-2.54_1x02_P2.54mm_Horizontal, symbol Connector:Screw_Terminal_01x02
- added SW5: External, Connector_Wuerth:Wuerth_WR-WTB_64800211622_1x02_P1.50mm_Vertical, symbol Switch:SW_SPST
- SW2, SW3, SW4: value B2B-XH-AM -> External
- renumbered PTC1 to F1
Connections:
- net +12V: now also J6.2 (Pin_2), SW5.2 (B); no longer F1.1, J2.1 (Pin_1), J3.1 (Pin_1)
- net GND: now also K1.5 (NC), K2.5 (NC); no longer K1.4 (NO), K2.4 (NO)
- net launch: now also R9.1, SW3.2 (B); no longer C1.1, K2.1 (Signal), R11.2, R9.2
- net safed_power: now also K2.4 (NO); no longer K2.5 (NC)
- net at F1.2: now also K1.4 (NO); no longer K1.5 (NC)
- new net battery: F1.1, J2.1 (Pin_1), J3.1 (Pin_1), J6.1 (Pin_1), SW5.1 (A)
- new net launch_sw: C1.1, K2.1 (Signal), R11.2, R9.2
Other:
- moved on the sheet: J2, J3
